File: avrboard.sch (EAGLE design)
At the start: 9 parts, among them IC1 MEGA48/88/168-AU, IC2 78L05SMD

Commit message: smaller fixes
Parts:
- added JP2, JP3: (no value), pinhead:PINHD-1X8
Connections:
- new net N$12: IC1.ADC7, JP2.8
- new net N$13: IC1.PD0(RXD/PCINT16), JP3.1
- new net N$14: IC1.PD1(TXD/PCINT17), JP3.2
- new net N$15: IC1.PD2(INT0/PCINT18), JP3.3
- new net N$16: IC1.PD3(INT1/OC2B/PCINT19), JP3.4
- new net N$17: IC1.PD4(T0/XCK/PCINT20), JP3.5
- new net N$18: IC1.PD5(T1/OC0B/PCINT21), JP3.6
- new net N$19: IC1.PD6(AIN0/OC0A/PCINT22), JP3.7
- new net N$2: IC1.PC0(ADC0/PCINT8), JP2.1
- new net N$20: IC1.PD7(AIN1/PCINT23), JP3.8
- new net N$3: IC1.PC1(ADC1/PCINT9), JP2.2
- new net N$4: IC1.PC2(ADC2/PCINT10), JP2.3
- new net N$5: IC1.PC3(ADC3/PCINT11), JP2.4
- new net N$6: IC1.PC4(ADC4/SDA/PCINT12), JP2.5
- new net N$7: IC1.PC5(ADC5/SCL/PCINT13), JP2.6
- new net N$8: IC1.ADC6, JP2.7
- net +5V: now also C1.1, C2.1, C3.1
- net GND: now also C1.2, C2.2, C3.2
Changed lines of the file:
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@@
 <part name="R1" library="resistor" deviceset="R-US_" device="R0805"/>
 <part name="P+5" library="supply1" deviceset="+5V" device=""/>
+<part name="P+6" library="supply1" deviceset="+5V" device=""/>
+<part name="GND4" library="supply1" deviceset="GND" device=""/>
+<part name="JP2" library="pinhead" deviceset="PINHD-1X8" device=""/>
+<part name="JP3" library="pinhead" deviceset="PINHD-1X8" device=""/>
 </parts>
 <sheets>
@@
 <instance part="R1" gate="G$1" x="22.86" y="139.7" rot="R90"/>
 <instance part="P+5" gate="1" x="22.86" y="152.4"/>
+<instance part="P+6" gate="1" x="20.32" y="53.34"/>
+<instance part="GND4" gate="1" x="20.32" y="17.78"/>
+<instance part="JP2" gate="A" x="119.38" y="121.92"/>
+<instance part="JP3" gate="A" x="137.16" y="99.06"/>
 </instances>
 <busses>
@@
 <pinref part="P+5" gate="1" pin="+5V"/>
 <wire x1="22.86" y1="144.78" x2="22.86" y2="149.86" width="0.1524" layer="91"/>
+</segment>
+<segment>
+<pinref part="C3" gate="G$1" pin="1"/>
+<wire x1="27.94" y1="40.64" x2="27.94" y2="45.72" width="0.1524" layer="91"/>
+<wire x1="27.94" y1="45.72" x2="20.32" y2="45.72" width="0.1524" layer="91"/>
+<pinref part="C1" gate="G$1" pin="1"/>
+<wire x1="20.32" y1="45.72" x2="12.7" y2="45.72" width="0.1524" layer="91"/>
+<wire x1="12.7" y1="45.72" x2="12.7" y2="40.64" width="0.1524" layer="91"/>
+<pinref part="C2" gate="G$1" pin="1"/>
+<wire x1="20.32" y1="40.64" x2="20.32" y2="45.72" width="0.1524" layer="91"/>
+<pinref part="P+6" gate="1" pin="+5V"/>
+<wire x1="20.32" y1="50.8" x2="20.32" y2="45.72" width="0.1524" layer="91"/>
 </segment>
 </net>
@@
 <pinref part="GND3" gate="1" pin="GND"/>
 </segment>
+<segment>
+<pinref part="C1" gate="G$1" pin="2"/>
+<wire x1="12.7" y1="33.02" x2="12.7" y2="25.4" width="0.1524" layer="91"/>
+<wire x1="12.7" y1="25.4" x2="20.32" y2="25.4" width="0.1524" layer="91"/>
+<pinref part="C3" gate="G$1" pin="2"/>
+<wire x1="20.32" y1="25.4" x2="27.94" y2="25.4" width="0.1524" layer="91"/>
+<wire x1="27.94" y1="25.4" x2="27.94" y2="33.02" width="0.1524" layer="91"/>
+<pinref part="C2" gate="G$1" pin="2"/>
+<wire x1="20.32" y1="33.02" x2="20.32" y2="25.4" width="0.1524" layer="91"/>
+<pinref part="GND4" gate="1" pin="GND"/>
+<wire x1="20.32" y1="20.32" x2="20.32" y2="25.4" width="0.1524" layer="91"/>
+</segment>
 </net>
 <net name="N$1" class="0">
@@
 </segment>
 </net>
+<net name="N$2" class="0">
+<segment>
+<pinref part="IC1" gate="1" pin="PC0(ADC0/PCINT8)"/>
+<pinref part="JP2" gate="A" pin="1"/>
+<wire x1="99.06" y1="132.08" x2="116.84" y2="132.08" width="0.1524" layer="91"/>
+</segment>
+</net>
+<net name="N$3" class="0">
+<segment>
+<pinref part="IC1" gate="1" pin="PC1(ADC1/PCINT9)"/>
+<pinref part="JP2" gate="A" pin="2"/>
+<wire x1="99.06" y1="129.54" x2="116.84" y2="129.54" width="0.1524" layer="91"/>
+</segment>
+</net>
+<net name="N$4" class="0">
+<segment>
+<pinref part="IC1" gate="1" pin="PC2(ADC2/PCINT10)"/>
+<pinref part="JP2" gate="A" pin="3"/>
+<wire x1="99.06" y1="127" x2="116.84" y2="127" width="0.1524" layer="91"/>
+</segment>
+</net>
+<net name="N$5" class="0">
+<segment>
+<pinref part="IC1" gate="1" pin="PC3(ADC3/PCINT11)"/>
+<pinref part="JP2" gate="A" pin="4"/>
+<wire x1="99.06" y1="124.46" x2="116.84" y2="124.46" width="0.1524" layer="91"/>
+</segment>
+</net>
+<net name="N$6" class="0">
+<segment>
+<pinref part="IC1" gate="1" pin="PC4(ADC4/SDA/PCINT12)"/>
+<pinref part="JP2" gate="A" pin="5"/>
+<wire x1="99.06" y1="121.92" x2="116.84" y2="121.92" width="0.1524" layer="91"/>
+</segment>
+</net>
+<net name="N$7" class="0">
+<segment>
+<pinref part="IC1" gate="1" pin="PC5(ADC5/SCL/PCINT13)"/>
+<pinref part="JP2" gate="A" pin="6"/>
+<wire x1="99.06" y1="119.38" x2="116.84" y2="119.38" width="0.1524" layer="91"/>
+</segment>
+</net>
+<net name="N$8" class="0">
+<segment>
+<pinref part="IC1" gate="1" pin="ADC6"/>
+<pinref part="JP2" gate="A" pin="7"/>
+<wire x1="99.06" y1="116.84" x2="116.84" y2="116.84" width="0.1524" layer="91"/>
+</segment>
+</net>
+<net name="N$12" class="0">
+<segment>
+<pinref part="IC1" gate="1" pin="ADC7"/>
+<pinref part="JP2" gate="A" pin="8"/>
+<wire x1="99.06" y1="114.3" x2="116.84" y2="114.3" width="0.1524" layer="91"/>
+</segment>
+</net>
+<net name="N$13" class="0">
+<segment>
+<pinref part="JP3" gate="A" pin="1"/>
+<pinref part="IC1" gate="1" pin="PD0(RXD/PCINT16)"/>
+<wire x1="134.62" y1="109.22" x2="99.06" y2="109.22" width="0.1524" layer="91"/>
+</segment>
+</net>
+<net name="N$14" class="0">
+<segment>
+<pinref part="JP3" gate="A" pin="2"/>
+<pinref part="IC1" gate="1" pin="PD1(TXD/PCINT17)"/>
+<wire x1="134.62" y1="106.68" x2="99.06" y2="106.68" width="0.1524" layer="91"/>
+</segment>
+</net>
+<net name="N$15" class="0">
+<segment>
+<pinref part="JP3" gate="A" pin="3"/>
+<pinref part="IC1" gate="1" pin="PD2(INT0/PCINT18)"/>
+<wire x1="134.62" y1="104.14" x2="99.06" y2="104.14" width="0.1524" layer="91"/>
+</segment>
+</net>
+<net name="N$16" class="0">
+<segment>
+<pinref part="JP3" gate="A" pin="4"/>
+<pinref part="IC1" gate="1" pin="PD3(INT1/OC2B/PCINT19)"/>
+<wire x1="134.62" y1="101.6" x2="99.06" y2="101.6" width="0.1524" layer="91"/>
+</segment>
+</net>
+<net name="N$17" class="0">
+<segment>
+<pinref part="JP3" gate="A" pin="5"/>
+<pinref part="IC1" gate="1" pin="PD4(T0/XCK/PCINT20)"/>
+<wire x1="134.62" y1="99.06" x2="99.06" y2="99.06" width="0.1524" layer="91"/>
+</segment>
+</net>
+<net name="N$18" class="0">
+<segment>
+<pinref part="JP3" gate="A" pin="6"/>
+<pinref part="IC1" gate="1" pin="PD5(T1/OC0B/PCINT21)"/>
+<wire x1="134.62" y1="96.52" x2="99.06" y2="96.52" width="0.1524" layer="91"/>
+</segment>
+</net>
+<net name="N$19" class="0">
+<segment>
+<pinref part="JP3" gate="A" pin="7"/>
+<pinref part="IC1" gate="1" pin="PD6(AIN0/OC0A/PCINT22)"/>
+<wire x1="134.62" y1="93.98" x2="99.06" y2="93.98" width="0.1524" layer="91"/>
+</segment>
+</net>
+<net name="N$20" class="0">
+<segment>
+<pinref part="JP3" gate="A" pin="8"/>
+<pinref part="IC1" gate="1" pin="PD7(AIN1/PCINT23)"/>
+<wire x1="134.62" y1="91.44" x2="99.06" y2="91.44" width="0.1524" layer="91"/>
+</segment>
+</net>

Commit message: updated readme, small fixes on schema
Parts:
- removed C3: 100nF, rcl:C-EUC0805
Connections:
- removed net N$1: IC1.AGND, IC1.GND@1, IC1.GND@2
- net +5V: no longer C3.1
- net GND: now also IC1.AGND, IC1.GND@1, IC1.GND@2; no longer C3.2
Changed lines of the file:
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@@
 <part name="C1" library="rcl" deviceset="C-EU" device="C0805" value="100nF"/>
 <part name="C2" library="rcl" deviceset="C-EU" device="C0805" value="100nF"/>
-<part name="C3" library="rcl" deviceset="C-EU" device="C0805" value="100nF"/>
 <part name="IC2" library="linear" deviceset="78L*SMD" device="" technology="05"/>
 <part name="C4" library="rcl" deviceset="C-EU" device="C0805" value="100nF"/>
@@
 <instance part="C1" gate="G$1" x="12.7" y="38.1"/>
 <instance part="C2" gate="G$1" x="20.32" y="38.1"/>
-<instance part="C3" gate="G$1" x="27.94" y="38.1"/>
 <instance part="IC2" gate="G$1" x="88.9" y="35.56"/>
 <instance part="C4" gate="G$1" x="111.76" y="33.02"/>
@@
 </segment>
 <segment>
-<pinref part="C3" gate="G$1" pin="1"/>
-<wire x1="27.94" y1="40.64" x2="27.94" y2="45.72" width="0.1524" layer="91"/>
-<wire x1="27.94" y1="45.72" x2="20.32" y2="45.72" width="0.1524" layer="91"/>
 <pinref part="C1" gate="G$1" pin="1"/>
 <wire x1="20.32" y1="45.72" x2="12.7" y2="45.72" width="0.1524" layer="91"/>
@@
 <wire x1="12.7" y1="33.02" x2="12.7" y2="25.4" width="0.1524" layer="91"/>
 <wire x1="12.7" y1="25.4" x2="20.32" y2="25.4" width="0.1524" layer="91"/>
-<pinref part="C3" gate="G$1" pin="2"/>
-<wire x1="20.32" y1="25.4" x2="27.94" y2="25.4" width="0.1524" layer="91"/>
-<wire x1="27.94" y1="25.4" x2="27.94" y2="33.02" width="0.1524" layer="91"/>
 <pinref part="C2" gate="G$1" pin="2"/>
 <wire x1="20.32" y1="33.02" x2="20.32" y2="25.4" width="0.1524" layer="91"/>
@@
 <wire x1="20.32" y1="20.32" x2="20.32" y2="25.4" width="0.1524" layer="91"/>
 </segment>
-</net>
-<net name="N$1" class="0">
 <segment>
 <pinref part="IC1" gate="1" pin="GND@2"/>
 <wire x1="38.1" y1="73.66" x2="27.94" y2="73.66" width="0.1524" layer="91"/>
-<wire x1="27.94" y1="73.66" x2="27.94" y2="68.58" width="0.1524" layer="91"/>
+<wire x1="27.94" y1="73.66" x2="27.94" y2="71.12" width="0.1524" layer="91"/>
 <pinref part="IC1" gate="1" pin="GND@1"/>
 <wire x1="38.1" y1="76.2" x2="27.94" y2="76.2" width="0.1524" layer="91"/>
@@
 <wire x1="38.1" y1="81.28" x2="27.94" y2="81.28" width="0.1524" layer="91"/>
 <wire x1="27.94" y1="81.28" x2="27.94" y2="76.2" width="0.1524" layer="91"/>
+<junction x="27.94" y="81.28"/>
+<junction x="27.94" y="76.2"/>
+<junction x="27.94" y="73.66"/>
 </segment>
 </net>
